File: CoordinateMeasurementLogicBoard.kicad_pcb (KiCad board)
At the start: 2 copper layers, 161 x 74 mm, 43 parts, among them J1 DE9_Receptacle_MountingHoles, J2 DE9_Receptacle_MountingHoles, J3 DE9_Receptacle_MountingHoles, J4 DE9_Receptacle_MountingHoles, J5 DE9_Receptacle_MountingHoles, Q1 BDP948, Q2 BC856, Q3 BC847, U1 AM2DS-0509SJZ

Commit message: optimized silkscreen; todo: added mounting holes, HTW logo and copyright
Routing:
- net GND: track 405.2 -> 0.00 mm
- net Net-(A1-D3): track 37.3 -> 40.0 mm
- net +5V: track 95.2 -> 97.3 mm
- net /Error_LED: track 31.8 -> 33.0 mm
- added copper zone on B.Cu, net GND
- added copper zone on F.Cu, net GND
Other:
- board text added: "ENC_ON"
- board text added: "ERROR"
- board text added: "PWR_OK"

Commit message: fix: R16 wasn't updated correctly
Parts:
- R16: value 10k -> 1k
Changed lines of the file:
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@@
 			)
 		)
-		(property "Value" "10k"
+		(property "Value" "1k"
 			(at 0 -1.4125 360)
 			(layer "B.Fab")
@@
 			)
 		)
-		(property "Reichelt.de" "SMD-0805 10,0K"
+		(property "Reichelt.de" "SMD-0805 1,0K"
 			(at 0 0 0)
 			(unlocked yes)

Commit message: ready; mounting holes; cosmetic
Parts:
- added H1: MountingHole_Pad, MountingHole:MountingHole_3.2mm_M3_Pad_Via, F.Cu at (33.0, 94.0)
- added H10: MountingHole_Pad, MountingHole:MountingHole_3.2mm_M3_Pad_Via, F.Cu at (153.0, 94.0)
- added H2: MountingHole_Pad, MountingHole:MountingHole_3.2mm_M3_Pad_Via, F.Cu at (183.0, 94.0)
- added H3: MountingHole_Pad, MountingHole:MountingHole_3.2mm_M3_Pad_Via, F.Cu at (33.0, 42.0)
- added H4: MountingHole_Pad, MountingHole:MountingHole_3.2mm_M3_Pad_Via, F.Cu at (100.0, 94.0)
- added H5: MountingHole_Pad, MountingHole:MountingHole_3.2mm_M3_Pad_Via, F.Cu at (183.0, 42.0)
- added H6: MountingHole_Pad, MountingHole:MountingHole_3.2mm_M3_Pad_Via, F.Cu at (93.0, 42.0)
- added H7: MountingHole_Pad, MountingHole:MountingHole_3.2mm_M3_Pad_Via, F.Cu at (153.0, 42.0)
- added H8: MountingHole_Pad, MountingHole:MountingHole_3.2mm_M3_Pad_Via, F.Cu at (123.0, 42.0)
- added H9: MountingHole_Pad, MountingHole:MountingHole_3.2mm_M3_Pad_Via, F.Cu at (63.0, 42.0)
- moved D6 4.00 mm to (176.5, 41.1)
- moved R10 4.00 mm to (168.5, 40.4)
- moved R9 4.00 mm to (172.5, 40.4)
- moved D4 2.50 mm to (113.5, 41.1)
- moved D5 2.50 mm to (145.5, 41.1)
- moved R5 2.50 mm to (109.5, 40.4)
- moved R6 2.50 mm to (105.5, 40.4)
- moved R7 2.50 mm to (141.5, 40.4)
- moved R8 2.50 mm to (137.5, 40.4)
Routing:
- net /PWR: track 258.8 -> 265.0 mm
- net /B4: track 128.3 -> 125.1 mm
- net /B2: track 76.1 -> 73.6 mm
- net /A2: track 76.3 -> 74.2 mm
- net /B3: track 100.1 -> 98.0 mm
- net /A4: track 128.9 -> 127.2 mm
- net Net-(J5-Pad3): track 8.64 -> 10.3 mm
- net /A3: track 102.0 -> 101.0 mm
- net Net-(J4-Pad3): track 8.72 -> 9.75 mm
- net Net-(J3-Pad3): track 8.57 -> 9.61 mm
- net Net-(D4-K): track 9.59 -> 8.59 mm
- net Net-(J5-Pad4): track 9.02 -> 9.79 mm
- net Net-(D5-K): track 9.45 -> 8.73 mm
Other:
- board text added: "Copyright (c) 2024 Stefan Helmert"

Commit message: replaced D-Sub-9 Connector
Parts:
- J1, J2, J3, J4, J5: footprint Connector_Dsub:DSUB-9_Female_Horizontal_P2.77x2.84mm_EdgePinOffset4.94mm_Housed_MountingHolesOffset7.48mm -> Connector_Dsub:DSUB-9_Socket_Horizontal_P2.77x2.84mm_EdgePinOffset7.70mm_Housed_MountingHolesOffset9.12mm
